Commit message: Created Gazebo simulation for robot

File: description/robot_core.xacro (robot description, xacro)
@@ -40,6 +40,12 @@
         </xacro:inertial_box>
     </link>
+    <!-- gazebo tag to also provide color in gazebo -->
+    <gazebo reference="chassis">
+        <material>
+            Gazebo/White
+        </material>
+    </gazebo>
     <!-- LEFT WHEEL LINK -->
-    <joint name="left_wheel_join" type="continuous">
+    <joint name="left_wheel_joint" type="continuous">
         <origin xyz="0 0.175 0" rpy="-${pi/2} 0.0 0.0"/>
         <parent link="base_link"/>
@@ -64,6 +70,11 @@
         </xacro:inertial_cylinder>
     </link>
+    <gazebo reference="left_wheel">
+        <material>
+            Gazebo/Blue
+        </material>
+    </gazebo>
     <!-- RIGHT WHEEL LINK -->
-    <joint name="right_wheel_join" type="continuous">
+    <joint name="right_wheel_joint" type="continuous">
         <origin xyz="0 -0.175 0" rpy="${pi/2} 0.0 0.0"/>
         <parent link="base_link"/>
@@ -88,6 +99,11 @@
         </xacro:inertial_cylinder>
     </link>
+    <gazebo reference="right_wheel">
+        <material>
+            Gazebo/Blue
+        </material>
+    </gazebo>
     <!-- CASTER WHEEL LINK  -->
-    <joint name="caster_wheel_jiont" type="fixed">
+    <joint name="caster_wheel_joint" type="fixed">
         <parent link="chassis"/>
         <child link="caster_wheel"/>
@@ -110,3 +126,10 @@
         </xacro:inertial_sphere>
     </link>
+    <gazebo reference="caster_wheel">
+        <material>
+            Gazebo/Black
+        </material>
+        <mu1 value="0.001" />
+        <mu2 value="0.001" />
+    </gazebo>
 </robot>
